File: hardware/Transmitter/2024.03.15_AVR_SCORE_BOARD_TX_v2/2024.03.15_AVR_SCORE_BOARD_TX_v2.kicad_pcb (KiCad board)
At the start: 2 copper layers, 47 parts, among them J1 Conn_01x10, J2 Conn_01x10, J3 Conn_01x05, J4 USB_B, Q1 BC817, SW1 SW_D1S+, SW10 D2S-, SW11 D2P+, SW12 D2P-, SW2 D1S-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

Commit message: Update label
Parts:
- SW6: value SW_H- -> SW_M+
